File: Eagle File/NRF52_Metal_Detector_v1.0/NRF52_Metal_Detector_v1.0.brd (EAGLE design)
At the start: 40.2 x 13.7 mm, 68 parts, among them IC1 ADA4841, IC2 MCP73831, IC3 TPS799_3.3V, IC4 MAX5048, IC5 TPS799_3.3V, IC7 TLV70235

Commit message: Update Eagle Files
Parts:
- C8: value 3n3 -> 10n
- C9: value 4n7 -> 10n
Changed lines of the file:
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@@
 <attribute name="VALUE" x="3.175" y="13.0175" size="1.27" layer="27" rot="R270"/>
 </element>
-<element name="C8" library="resistor" package="C1206" value="3n3" x="30.4712" y="1.2553" smashed="yes" rot="MR0">
+<element name="C8" library="resistor" package="C1206" value="10n" x="30.4712" y="1.2553" smashed="yes" rot="MR0">
 <attribute name="NAME" x="31.5825" y="0.6203" size="1.27" layer="26" rot="MR0"/>
 <attribute name="VALUE" x="32.3762" y="0.6203" size="1.27" layer="28" rot="MR0"/>
@@
 <attribute name="VALUE" x="23.173" y="4.749" size="1.27" layer="28" rot="MR270"/>
 </element>
-<element name="C9" library="resistor" package="C1206" value="4n7" x="30.4712" y="3.1591" smashed="yes" rot="MR0">
+<element name="C9" library="resistor" package="C1206" value="10n" x="30.4712" y="3.1591" smashed="yes" rot="MR0">
 <attribute name="NAME" x="31.5825" y="2.5241" size="1.27" layer="26" rot="MR0"/>
 <attribute name="VALUE" x="31.7412" y="0.6191" size="1.27" layer="28" rot="MR0"/>
