File: Eagle File/NRF52_Metal_Detector_v1.0/NRF52_Metal_Detector_v1.0.sch (EAGLE design)
At the start: 68 parts, among them IC1 ADA4841, IC2 MCP73831, IC3 TPS799_3.3V, IC4 MAX5048, IC5 TPS799_3.3V, IC7 TLV70235

Commit message: Update Eagle Files
Parts:
- C8: value 3n3 -> 10n
- C9: value 4n7 -> 10n
Changed lines of the file:
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@@
 <part name="R1" library="resistor" deviceset="R-EU_" device="R0805" value="4k7"/>
 <part name="GND5" library="supply1" deviceset="GND" device=""/>
-<part name="C8" library="resistor" deviceset="C-EU" device="C1206" value="3n3"/>
+<part name="C8" library="resistor" deviceset="C-EU" device="C1206" value="10n"/>
 <part name="GND7" library="supply1" deviceset="GND" device=""/>
 <part name="C4" library="resistor" deviceset="C-EU" device="C1206" value="1u"/>
@@
 <part name="R3" library="resistor" deviceset="R-EU_" device="R0805" value="3k3"/>
 <part name="C23" library="resistor" deviceset="C-EU" device="C1206" value="22u"/>
-<part name="C9" library="resistor" deviceset="C-EU" device="C1206" value="4n7"/>
+<part name="C9" library="resistor" deviceset="C-EU" device="C1206" value="10n"/>
 <part name="R10" library="resistor" deviceset="R-EU_" device="R0805" value="47r"/>
 <part name="+3V3" library="supply1" deviceset="+3V3" device="" value="Rx_VCC"/>
